Commit message: path issues correction

File: assets/turtlebot3_waffle_pi/urdf/turtlebot3_waffle_pi.urdf (robot description, URDF)
Before this commit: robot turtlebot3_waffle_pi, 11 links, 10 joints
Links:
- link base_link: geometry collision box size=0.266 0.266 0.094; visual mesh filename=current_path/assets/turtlebot3_waffle_pi/meshes/bases/waffl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 scale=0.001 0.001 0.001
- link base_scan: geometry collision cylinder length=0.0315 radius=0.055; visual mesh filename=current_path/assets/turtlebot3_waffle_pi/meshes/sensors/lds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 scale=0.001 0.001 0.001
- link wheel_left_link: geometry collision cylinder length=0.018 radius=0.033; visual mesh filename=current_path/assets/turtlebot3_waffle_pi/meshes/wheels/left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 scale=0.001 0.001 0.001
- link wheel_right_link: geometry collision cylinder length=0.018 radius=0.033; visual mesh filename=current_path/assets/turtlebot3_waffle_pi/meshes/wheels/righ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 scale=0.001 0.001 0.001
